Commit message: 推定の安定性を向上

File: src/description/urdf/robot.urdf (robot description, URDF)
Before this commit: robot robot, 7 links, 6 joints
Joints:
- joint BL_joint: limit lower=-1000000000000 upper=1000000000000 effort=2000 velocity=80.0 -> lower=-1000000000000 upper=1000000000000 effort=2000 velocity=20.0
- joint BR_joint: limit lower=-1000000000000 upper=1000000000000 effort=2000 velocity=80.0 -> lower=-1000000000000 upper=1000000000000 effort=2000 velocity=20.0
- joint FL_joint: limit lower=-1000000000000 upper=1000000000000 effort=2000 velocity=80.0 -> lower=-1000000000000 upper=1000000000000 effort=2000 velocity=20.0
- joint FR_joint: limit lower=-1000000000000 upper=1000000000000 effort=2000 velocity=80.0 -> lower=-1000000000000 upper=1000000000000 effort=2000 velocity=20.0
