Commit message: 一から作り直し開始

File: src/bring_up/urdf/robot.urdf (robot description, URDF)
Before this commit: robot robot, 7 links, 6 joints
Links:
- link BL_wheel: mass 1.5 -> 1.0; geometry collision cylinder length=0.04 radius=0.1; visual cylinder length=0.04 radius=0.1
- link BR_wheel: mass 1.5 -> 1.0; geometry collision cylinder length=0.04 radius=0.1; visual cylinder length=0.04 radius=0.1
- link FL_wheel: mass 1.5 -> 1.0; geometry collision cylinder length=0.04 radius=0.1; visual cylinder length=0.04 radius=0.1
- link FR_wheel: mass 1.5 -> 1.0; geometry collision cylinder length=0.04 radius=0.1; visual cylinder length=0.04 radius=0.1
- link robot_base: mass 30.0 -> 26.0; geometry collision cylinder length=0.1 radius=0.4; visual cylinder length=0.1 radius=0.4
Joints:
- joint BL_joint: limit lower=-1000000000000 upper=1000000000000 effort=2000 velocity=20.0 -> lower=-1000000000000 upper=1000000000000 effort=2000 velocity=40.0; origin xyz=-0.25 0.25 0.0 rpy=1.571 0 -2.356125 -> xyz=-0.282842712 0.282842712 0.0 rpy=1.571 0 -2.356125
- joint BR_joint: limit lower=-1000000000000 upper=1000000000000 effort=2000 velocity=20.0 -> lower=-1000000000000 upper=1000000000000 effort=2000 velocity=40.0; origin xyz=-0.25 -0.25 0.0 rpy=1.571 0 -0.785375 -> xyz=-0.282842712 -0.282842712 0.0 rpy=1.571 0 -0.785375
- joint FL_joint: limit lower=-1000000000000 upper=1000000000000 effort=2000 velocity=20.0 -> lower=-1000000000000 upper=1000000000000 effort=2000 velocity=40.0; origin xyz=0.25 0.25 0.0 rpy=1.571 0 2.356125 -> xyz=0.282842712 0.282842712 0.0 rpy=1.571 0 2.356125
- joint FR_joint: limit lower=-1000000000000 upper=1000000000000 effort=2000 velocity=20.0 -> lower=-1000000000000 upper=1000000000000 effort=2000 velocity=40.0; origin xyz=0.25 -0.25 0.0 rpy=1.571 0 0.785375 -> xyz=0.282842712 -0.282842712 0.0 rpy=1.571 0 0.785375
- joint left_lidar_joint: origin xyz=0.0 0.35 -0.008 rpy=0.0 0.0 1.571 -> xyz=0.0 0.4 -0.06 rpy=0.0 0.0 1.571
- joint right_lidar_joint: origin xyz=0.0 -0.35 -0.008 rpy=0.0 0.0 -1.571 -> xyz=0.0 -0.4 -0.06 rpy=0.0 0.0 -1.571

Commit message: 20250703

File: src/bring_up/urdf/robot.urdf (robot description, URDF)
Before this commit: robot robot, 7 links, 6 joints
Links:
- link BL_wheel: geometry collision cylinder length=0.1 radius=0.10; visual cylinder length=0.1 radius=0.10
- link BR_wheel: geometry collision cylinder length=0.1 radius=0.10; visual cylinder length=0.1 radius=0.10
- link FL_wheel: geometry collision cylinder length=0.1 radius=0.10; visual cylinder length=0.1 radius=0.10
- link FR_wheel: geometry collision cylinder length=0.1 radius=0.10; visual cylinder length=0.1 radius=0.10
